File: carte_thyristor_triac/sae_four_manip_triac/SAE_four_manip_triac.kicad_sch (KiCad schematic)
At the start: 23 parts, among them J2 Conn_01x02_Pin, J3 Conn_01x02_Pin, J4 SWEB_8094_Au___SW, J5 Jack-DC, J5 SWEB_8094_Au___SW, Q1 BT136-600, U4 L78L05_TO92, U5 4N35, U6 MOC3022M, U7 MOC3061M

Commit message: update triac et librairies
Parts:
- removed J4, J5: SWEB_8094_Au___SW, SWEB8094AuSW, symbol douille:SWEB_8094_Au___SW
- added J1: SWEB_8094_Au___SW, SamacSys_Parts:douille_4mm_SWEB_8094_rouge, symbol SamacSys_Parts:SWEB_8094_Au___SW
- added J4: SWEB_8094_Au___SW, SamacSys_Parts:douille_4mm_SWEB_8094_noire, symbol SamacSys_Parts:SWEB_8094_Au___SW
- C2: footprint Capacitor_THT:C_Axial_L5.1mm_D3.1mm_P7.50mm_Horizontal -> Capacitor_THT:C_Rect_L4.6mm_W3.8mm_P2.50mm_MKS02_FKP02
- J2, J3: footprint (none) -> Connector_PinHeader_2.54mm:PinHeader_1x02_P2.54mm_Vertical
- J5: footprint Connector_BarrelJack:BarrelJack_GCT_DCJ200-10-A_Horizontal -> SamacSys_Parts:BarrelJack_GCT_DCJ200-10-A_Horizontal_3D
- R1, R3, R4, R5, R6: footprint Resistor_THT:R_Bare_Metal_Element_L12.4mm_W4.8mm_P11.40mm -> Resistor_THT:R_Axial_DIN0207_L6.3mm_D2.5mm_P10.16mm_Horizontal
Connections:
- net GND: now also J3.2 (Pin_2), J3.2 (Pin_2), J4.1, J4.2, J4.3, J4.4
- net at D1.1 (K), D3.2 (A), Q1.1 (A1): now also J1.1, J1.2, J1.3, J1.4
